Commit message: add chasis to 280jn urdf

File: mycobot_description/urdf/280jn/mycobot_urdf.urdf (robot description, URDF)
Before this commit: robot firefighter, 7 links, 6 joints
Links:
- added link chasis; collision mesh filename=package://mycobot_description/urdf/280jn/chasis.obj; visual mesh filename=package://mycobot_description/urdf/280jn/chasis.obj
Joints:
- added joint joint1_to_chasis: type fixed, parent chasis, child joint1
